File: 286_to_bboard.kicad_sch (KiCad schematic)
At the start: 28 parts, among them J1 Conn_01x30, J2 Conn_01x30, J3 Conn_01x02, U1 74HC240

Commit message: finalize initial design
Parts:
- added C6: C, Capacitor_SMD:C_0805_2012Metric_Pad1.18x1.45mm_HandSolder, symbol Device:C
- C1, C2, C3, C4: footprint Capacitor_SMD:C_0805_2012Metric -> Capacitor_SMD:C_0805_2012Metric_Pad1.18x1.45mm_HandSolder
- C5: footprint Capacitor_SMD:C_0402_1005Metric -> Capacitor_SMD:C_0402_1005Metric_Pad0.74x0.62mm_HandSolder
- J1, J2: footprint Connector_PinSocket_2.54mm:PinSocket_1x30_P2.54mm_Vertical_SMD_Pin1Left -> Connector_PinHeader_2.54mm:PinHeader_1x30_P2.54mm_Vertical_SMD_Pin1Left
- R9: footprint Resistor_SMD:R_0402_1005Metric -> Resistor_SMD:R_0402_1005Metric_Pad0.72x0.64mm_HandSolder
Connections:
- net CLK: now also J1.27 (Pin_27); no longer J1.28 (Pin_28)
- net GND: now also J1.29 (Pin_29), J2.6 (Pin_6), C6.2; no longer J1.27 (Pin_27), J2.5 (Pin_5)
- net M/~{IO}: now also J1.5 (Pin_5); no longer J1.7 (Pin_7)
- net RESET: now also J1.28 (Pin_28); no longer J1.30 (Pin_30)
- net VCC: now also C1.1, J1.30 (Pin_30); no longer J1.29 (Pin_29), J2.6 (Pin_6)
- net ~{BHE}: now also J1.6 (Pin_6); no longer J1.8 (Pin_8)
- net ~{READY}: now also J2.5 (Pin_5)
- net ~{S0}: now also J1.8 (Pin_8); no longer J1.6 (Pin_6)
- net ~{S1}: now also J1.7 (Pin_7); no longer J1.5 (Pin_5)
- net at UA1.52 (CAP): now also C6.1; no longer C1.1
Other:
- moved on the sheet: C1, C2, C3, C4

Commit message: small revisions
Parts:
- C1, C3, C4, C5: value C -> 100nf
- C2: value C -> 10uf
- C6: value C -> 47nf
- U1: value 74HC240 -> 74HC244; symbol 74xx:74HC240 -> 74xx:74HC244
Other:
- moved on the sheet: C1, C2, C3, C4, C5
